File: rodentdbs.kicad_pcb (KiCad board)
At the start: 4 copper layers, 30.5 x 30.5 mm, 35 parts, among them IC1 MAX1724EZK50+T, J2 ELECTRODE, J3 BATTERY, J4 MECHANICAL, J6 Program, U2 CY8C4247LQI-BL493, Y1 ECS-.327-9-34B-C-TR, Y2 ECS-240-8-33-RWY-TR

Commit message: Fixed capacitor layout error in Rev 1.0 design
Parts:
- removed C17: 10 uF, Capacitor_SMD:C_0603_1608Metric
- removed J6: Program, Connector_PinHeader_1.27mm:PinHeader_1x05_P1.27mm_Vertical
- added J1: Program, Connector_PinHeader_1.27mm:PinHeader_1x05_P1.27mm_Vertical, F.Cu at (150.2, 123.0)
- AE1: value 2450AT42B100E -> Ant
- C14: value C -> 10uF; footprint Capacitor_SMD:C_0402_1005Metric -> Capacitor_SMD:C_0603_1608Metric; moved to B.Cu
- C15: value C -> 1.5pF
- C8: value 1.3uF -> 1.0uF
- D1: value LED -> RED LED
- D2: value LED -> GREEN LED
- L2: value L -> 3.5 nH
- moved C14 16.9 mm to (133.2, 126.4), turned to 0 degrees
- moved C15 1.78 mm to (146.1, 115.6), turned to 63.43 degrees
- moved L2 1.14 mm to (144.8, 114.3)
Connections:
- C14 pad 1: /rodentdbs_1/ANT -> /rodentdbs_1/VDDA
- C14 pad 2: Net-(AE1-FEED) -> GND
- C15 pad 1: GND -> /rodentdbs_1/ANT
- L2 pad 1: /rodentdbs_1/ANT -> Net-(AE1-FEED)
Routing:
- net /rodentdbs_1/VDDA: track 45.3 -> 46.9 mm
- net /rodentdbs_1/ANT: track 14.3 -> 12.9 mm
- net GND: vias 45 -> 44
- net /rodentdbs_1/SWDCLK: vias 1 -> 2
